Commit message: new base urdf

File: fusion_360_export/base_export_description/urdf/base_export.xacro (robot description, xacro)
@@ -6,7 +6,7 @@
 <link name="base_link">
   <inertial>
-    <origin rpy="0 0 0" xyz="-0.3482345382752994 -0.27514770765017643 0.19695481512469734"/>
-    <mass value="155.853533341384"/>
-    <inertia ixx="24.527524" ixy="0.013804" ixz="-0.002107" iyy="13.832614" iyz="-2.456883" izz="21.12491"/>
+    <origin rpy="0 0 0" xyz="0.004639774814419823 1.4771468453425644e-05 0.22530002486564402"/>
+    <mass value="90.2870635836035"/>
+    <inertia ixx="10.456164" ixy="1.4e-05" ixz="-0.360506" iyy="16.958749" iyz="0.000256" izz="18.430844"/>
   </inertial>
   <visual>
@@ -24,12 +24,52 @@
   </collision>
 </link>
+<link name="Nema34_1">
+  <inertial>
+    <origin rpy="0 0 0" xyz="-0.0006437918942043819 0.09929626309979397 0.0006420516696096987"/>
+    <mass value="6.652128143458834"/>
+    <inertia ixx="0.012865" ixy="1e-06" ixz="-0.0" iyy="0.007046" iyz="0.0" izz="0.012866"/>
+  </inertial>
+  <visual>
+    <origin rpy="0 0 0" xyz="-0.394801 0.200178 -0.033729"/>
+    <geometry>
+      <mesh filename="package://base_export_description/meshes/Nema34_1.stl" scale="0.001 0.001 0.001"/>
+    </geometry>
+    <material name="silver"/>
+  </visual>
+  <collision>
+    <origin rpy="0 0 0" xyz="-0.394801 0.200178 -0.033729"/>
+    <geometry>
+      <mesh filename="package://base_export_description/meshes/Nema34_1.stl" scale="0.001 0.001 0.001"/>
+    </geometry>
+  </collision>
+</link>
+<link name="Nema34__1__1">
+  <inertial>
+    <origin rpy="0 0 0" xyz="0.0006436418750596085 -0.09929646649528492 0.0006420516696081444"/>
+    <mass value="6.652128143458834"/>
+    <inertia ixx="0.012865" ixy="1e-06" ixz="0.0" iyy="0.007046" iyz="-0.0" izz="0.012866"/>
+  </inertial>
+  <visual>
+    <origin rpy="0 0 0" xyz="-0.394579 -0.200822 -0.033729"/>
+    <geometry>
+      <mesh filename="package://base_export_description/meshes/Nema34__1__1.stl" scale="0.001 0.001 0.001"/>
+    </geometry>
+    <material name="silver"/>
+  </visual>
+  <collision>
+    <origin rpy="0 0 0" xyz="-0.394579 -0.200822 -0.033729"/>
+    <geometry>
+      <mesh filename="package://base_export_description/meshes/Nema34__1__1.stl" scale="0.001 0.001 0.001"/>
+    </geometry>
+  </collision>
+</link>
 <link name="Double_Wheel__Thin__v11_v3_1">
   <inertial>
-    <origin rpy="0 0 0" xyz="-0.027863208093181154 -6.429566710543232e-11 5.495589618411427e-10"/>
+    <origin rpy="0 0 0" xyz="-3.5966591938052517e-07 0.027463106395432424 3.514880312152635e-07"/>
     <mass value="3.260021800926923"/>
-    <inertia ixx="0.009383" ixy="0.0" ixz="-0.0" iyy="0.005841" iyz="-0.0" izz="0.005841"/>
+    <inertia ixx="0.005841" ixy="-0.0" ixz="-0.0" iyy="0.009383" iyz="0.0" izz="0.005841"/>
   </inertial>
   <visual>
-    <origin rpy="0 0 0" xyz="-0.024 -0.0 0.0"/>
+    <origin rpy="0 0 0" xyz="-0.394801 0.390178 -0.033729"/>
     <geometry>
       <mesh filename="package://base_export_description/meshes/Double_Wheel__Thin__v11_v3_1.stl" scale="0.001 0.001 0.001"/>
@@ -38,5 +78,5 @@
   </visual>
   <collision>
-    <origin rpy="0 0 0" xyz="-0.024 -0.0 0.0"/>
+    <origin rpy="0 0 0" xyz="-0.394801 0.390178 -0.033729"/>
     <geometry>
       <mesh filename="package://base_export_description/meshes/Double_Wheel__Thin__v11_v3_1.stl" scale="0.001 0.001 0.001"/>
@@ -46,10 +86,10 @@
 <link name="Double_Wheel__Thin__v11_v3__1__1">
   <inertial>
-    <origin rpy="0 0 0" xyz="0.027863044321248198 1.7510568478515984e-07 5.493755826604987e-10"/>
+    <origin rpy="0 0 0" xyz="2.096467722756401e-07 -0.02746330979092404 3.5148803025075726e-07"/>
     <mass value="3.260021800926923"/>
-    <inertia ixx="0.009383" ixy="0.0" ixz="0.0" iyy="0.005841" iyz="0.0" izz="0.005841"/>
+    <inertia ixx="0.005841" ixy="-0.0" ixz="0.0" iyy="0.009383" iyz="-0.0" izz="0.005841"/>
   </inertial>
   <visual>
-    <origin rpy="0 0 0" xyz="0.72108 0.000192 0.0"/>
+    <origin rpy="0 0 0" xyz="-0.394579 -0.390822 -0.033729"/>
     <geometry>
       <mesh filename="package://base_export_description/meshes/Double_Wheel__Thin__v11_v3__1__1.stl" scale="0.001 0.001 0.001"/>
@@ -58,5 +98,5 @@
   </visual>
   <collision>
-    <origin rpy="0 0 0" xyz="0.72108 0.000192 0.0"/>
+    <origin rpy="0 0 0" xyz="-0.394579 -0.390822 -0.033729"/>
     <geometry>
       <mesh filename="package://base_export_description/meshes/Double_Wheel__Thin__v11_v3__1__1.stl" scale="0.001 0.001 0.001"/>
@@ -66,10 +106,10 @@
 <link name="Double_Wheel__Thin__v11_v3__2__1">
   <inertial>
-    <origin rpy="0 0 0" xyz="-0.027863208093183288 -6.429579091360438e-11 5.495594355558359e-10"/>
+    <origin rpy="0 0 0" xyz="2.0964677233115125e-07 -0.027463309790926815 3.51488031312408e-07"/>
     <mass value="3.260021800926923"/>
-    <inertia ixx="0.009383" ixy="0.0" ixz="-0.0" iyy="0.005841" iyz="-0.0" izz="0.005841"/>
+    <inertia ixx="0.005841" ixy="-0.0" ixz="0.0" iyy="0.009383" iyz="-0.0" izz="0.005841"/>
   </inertial>
   <visual>
-    <origin rpy="0 0 0" xyz="-0.024 0.665 -0.0"/>
+    <origin rpy="0 0 0" xyz="0.395421 -0.390822 -0.033729"/>
     <geometry>
       <mesh filename="package://base_export_description/meshes/Double_Wheel__Thin__v11_v3__2__1.stl" scale="0.001 0.001 0.001"/>
@@ -78,5 +118,5 @@
   </visual>
   <collision>
-    <origin rpy="0 0 0" xyz="-0.024 0.665 -0.0"/>
+    <origin rpy="0 0 0" xyz="0.395421 -0.390822 -0.033729"/>
     <geometry>
       <mesh filename="package://base_export_description/meshes/Double_Wheel__Thin__v11_v3__2__1.stl" scale="0.001 0.001 0.001"/>
@@ -86,10 +126,10 @@
 <link name="Double_Wheel__Thin__v11_v3__3__1">
   <inertial>
-    <origin rpy="0 0 0" xyz="0.027863044321161157 1.7510568439682572e-07 5.495610077369151e-10"/>
+    <origin rpy="0 0 0" xyz="-3.596659204907482e-07 0.02746310639543431 3.514880312152635e-07"/>
     <mass value="3.260021800926923"/>
-    <inertia ixx="0.009383" ixy="0.0" ixz="0.0" iyy="0.005841" iyz="0.0" izz="0.005841"/>
+    <inertia ixx="0.005841" ixy="-0.0" ixz="-0.0" iyy="0.009383" iyz="0.0" izz="0.005841"/>
   </inertial>
   <visual>
-    <origin rpy="0 0 0" xyz="0.72108 0.665192 -0.0"/>
+    <origin rpy="0 0 0" xyz="0.395199 0.390178 -0.033729"/>
     <geometry>
       <mesh filename="package://base_export_description/meshes/Double_Wheel__Thin__v11_v3__3__1.stl" scale="0.001 0.001 0.001"/>
@@ -98,5 +138,5 @@
   </visual>
   <collision>
-    <origin rpy="0 0 0" xyz="0.72108 0.665192 -0.0"/>
+    <origin rpy="0 0 0" xyz="0.395199 0.390178 -0.033729"/>
     <geometry>
       <mesh filename="package://base_export_description/meshes/Double_Wheel__Thin__v11_v3__3__1.stl" scale="0.001 0.001 0.001"/>
@@ -104,27 +144,37 @@
   </collision>
 </link>
-<joint name="Rev26" type="continuous">
-  <origin rpy="0 0 0" xyz="0.024 0.0 0.0"/>
+<joint name="Rigid9" type="fixed">
+  <origin rpy="0 0 0" xyz="0.394801 -0.200178 0.033729"/>
+  <parent link="base_link"/>
+  <child link="Nema34_1"/>
+</joint>
+<joint name="Rigid10" type="fixed">
+  <origin rpy="0 0 0" xyz="0.394579 0.200822 0.033729"/>
+  <parent link="base_link"/>
+  <child link="Nema34__1__1"/>
+</joint>
+<joint name="Rev11" type="continuous">
+  <origin rpy="0 0 0" xyz="0.394801 -0.390178 0.033729"/>
   <parent link="base_link"/>
   <child link="Double_Wheel__Thin__v11_v3_1"/>
-  <axis xyz="-1.0 -0.0 0.0"/>
+  <axis xyz="0.0 1.0 -0.0"/>
 </joint>
-<joint name="Rev27" type="continuous">
-  <origin rpy="0 0 0" xyz="-0.72108 -0.000192 0.0"/>
+<joint name="Rev12" type="continuous">
+  <origin rpy="0 0 0" xyz="0.394579 0.390822 0.033729"/>
   <parent link="base_link"/>
   <child link="Double_Wheel__Thin__v11_v3__1__1"/>
-  <axis xyz="1.0 -0.0 -0.0"/>
+  <axis xyz="0.0 -1.0 -0.0"/>
 </joint>
-<joint name="Rev28" type="continuous">
-  <origin rpy="0 0 0" xyz="0.024 -0.665 0.0"/>
+<joint name="Rev13" type="continuous">
+  <origin rpy="0 0 0" xyz="-0.395421 0.390822 0.033729"/>
   <parent link="base_link"/>
   <child link="Double_Wheel__Thin__v11_v3__2__1"/>
-  <axis xyz="-1.0 -0.0 -0.0"/>
+  <axis xyz="0.0 -1.0 -0.0"/>
 </joint>
-<joint name="Rev29" type="continuous">
-  <origin rpy="0 0 0" xyz="-0.72108 -0.665192 0.0"/>
+<joint name="Rev14" type="continuous">
+  <origin rpy="0 0 0" xyz="-0.395199 -0.390178 0.033729"/>
   <parent link="base_link"/>
   <child link="Double_Wheel__Thin__v11_v3__3__1"/>
-  <axis xyz="1.0 -0.0 -0.0"/>
+  <axis xyz="0.0 1.0 -0.0"/>
 </joint>
 </robot>
