Commit message: gripper added

File: fusion_360_export/Robot_description/urdf/Robot.xacro (robot description, xacro)
@@ -364,4 +364,84 @@
   </collision>
 </link>
+<link name="gripper_export_v2_1">
+  <inertial>
+    <origin rpy="0 0 0" xyz="0.036736557885818755 8.738047091449985e-10 4.869867763490632e-07"/>
+    <mass value="1.1315792783817065"/>
+    <inertia ixx="0.001318" ixy="-0.0" ixz="-0.0" iyy="0.001126" iyz="0.0" izz="0.001126"/>
+  </inertial>
+  <visual>
+    <origin rpy="0 0 0" xyz="-1.62405 0.02848 -0.820847"/>
+    <geometry>
+      <mesh filename="package://Robot_description/meshes/gripper_export_v2_1.stl" scale="0.001 0.001 0.001"/>
+    </geometry>
+    <material name="silver"/>
+  </visual>
+  <collision>
+    <origin rpy="0 0 0" xyz="-1.62405 0.02848 -0.820847"/>
+    <geometry>
+      <mesh filename="package://Robot_description/meshes/gripper_export_v2_1.stl" scale="0.001 0.001 0.001"/>
+    </geometry>
+  </collision>
+</link>
+<link name="EndEffector_v1_1">
+  <inertial>
+    <origin rpy="0 0 0" xyz="0.022979968590663757 3.2830825211216386e-10 0.004865820638522034"/>
+    <mass value="0.07511526055866109"/>
+    <inertia ixx="3e-06" ixy="-0.0" ixz="-0.0" iyy="1.7e-05" iyz="0.0" izz="1.8e-05"/>
+  </inertial>
+  <visual>
+    <origin rpy="0 0 0" xyz="-1.70855 0.02848 -0.853347"/>
+    <geometry>
+      <mesh filename="package://Robot_description/meshes/EndEffector_v1_1.stl" scale="0.001 0.001 0.001"/>
+    </geometry>
+    <material name="silver"/>
+  </visual>
+  <collision>
+    <origin rpy="0 0 0" xyz="-1.70855 0.02848 -0.853347"/>
+    <geometry>
+      <mesh filename="package://Robot_description/meshes/EndEffector_v1_1.stl" scale="0.001 0.001 0.001"/>
+    </geometry>
+  </collision>
+</link>
+<link name="EndEffector_v1__1__1">
+  <inertial>
+    <origin rpy="0 0 0" xyz="0.02297996859066398 -0.004213328299858453 -0.0024321799597640803"/>
+    <mass value="0.07511526055866109"/>
+    <inertia ixx="3e-06" ixy="0.0" ixz="0.0" iyy="1.8e-05" iyz="0.0" izz="1.8e-05"/>
+  </inertial>
+  <visual>
+    <origin rpy="0 0 0" xyz="-1.70855 0.056626 -0.804597"/>
+    <geometry>
+      <mesh filename="package://Robot_description/meshes/EndEffector_v1__1__1.stl" scale="0.001 0.001 0.001"/>
+    </geometry>
+    <material name="silver"/>
+  </visual>
+  <collision>
+    <origin rpy="0 0 0" xyz="-1.70855 0.056626 -0.804597"/>
+    <geometry>
+      <mesh filename="package://Robot_description/meshes/EndEffector_v1__1__1.stl" scale="0.001 0.001 0.001"/>
+    </geometry>
+  </collision>
+</link>
+<link name="EndEffector_v1__2__1">
+  <inertial>
+    <origin rpy="0 0 0" xyz="0.02297996859066398 0.004213328102255326 -0.002432180302022635"/>
+    <mass value="0.07511526055866109"/>
+    <inertia ixx="3e-06" ixy="-0.0" ixz="0.0" iyy="1.8e-05" iyz="-0.0" izz="1.8e-05"/>
+  </inertial>
+  <visual>
+    <origin rpy="0 0 0" xyz="-1.70855 0.000334 -0.804597"/>
+    <geometry>
+      <mesh filename="package://Robot_description/meshes/EndEffector_v1__2__1.stl" scale="0.001 0.001 0.001"/>
+    </geometry>
+    <material name="silver"/>
+  </visual>
+  <collision>
+    <origin rpy="0 0 0" xyz="-1.70855 0.000334 -0.804597"/>
+    <geometry>
+      <mesh filename="package://Robot_description/meshes/EndEffector_v1__2__1.stl" scale="0.001 0.001 0.001"/>
+    </geometry>
+  </collision>
+</link>
 <joint name="Rigid1" type="fixed">
   <origin rpy="0 0 0" xyz="0.51905 0.0 0.555847"/>
@@ -458,3 +538,26 @@
   <child link="Intel_RealSense_D435_v3_1"/>
 </joint>
+<joint name="Rigid18" type="fixed">
+  <origin rpy="0 0 0" xyz="0.05 0.04 0.0"/>
+  <parent link="joint_end_v3_1"/>
+  <child link="gripper_export_v2_1"/>
+</joint>
+<joint name="Rev19" type="continuous">
+  <origin rpy="0 0 0" xyz="0.0845 0.0 0.0325"/>
+  <parent link="gripper_export_v2_1"/>
+  <child link="EndEffector_v1_1"/>
+  <axis xyz="0.0 -1.0 0.0"/>
+</joint>
+<joint name="Rev20" type="continuous">
+  <origin rpy="0 0 0" xyz="0.0845 -0.028146 -0.01625"/>
+  <parent link="gripper_export_v2_1"/>
+  <child link="EndEffector_v1__1__1"/>
+  <axis xyz="0.0 0.5 -0.866025"/>
+</joint>
+<joint name="Rev21" type="continuous">
+  <origin rpy="0 0 0" xyz="0.0845 0.028146 -0.01625"/>
+  <parent link="gripper_export_v2_1"/>
+  <child link="EndEffector_v1__2__1"/>
+  <axis xyz="-0.0 0.5 0.866025"/>
+</joint>
 </robot>

File: fusion_360_export/arm_export_description/urdf/arm_export.xacro (robot description, xacro)
@@ -6,7 +6,7 @@
 <link name="base_link">
   <inertial>
-    <origin rpy="0 0 0" xyz="3.604012374114634e-17 0.019362619281988985 0.06375532936051907"/>
-    <mass value="2.725446463418606"/>
-    <inertia ixx="0.021529" ixy="0.0" ixz="0.0" iyy="0.015666" iyz="-0.002614" izz="0.028323"/>
+    <origin rpy="0 0 0" xyz="-9.029061793754004e-14 0.016476818393225144 0.07021749351752887"/>
+    <mass value="2.9829690964186772"/>
+    <inertia ixx="0.024074" ixy="-0.0" ixz="-0.0" iyy="0.017973" iyz="-0.002884" izz="0.02919"/>
   </inertial>
   <visual>
@@ -24,92 +24,52 @@
   </collision>
 </link>
+<link name="base_turnable_v14_1">
+  <inertial>
+    <origin rpy="0 0 0" xyz="-0.02993448375707213 0.004673714897230209 0.1005386168410774"/>
+    <mass value="7.350921302447738"/>
+    <inertia ixx="0.39669" ixy="-0.000566" ixz="0.055433" iyy="0.40707" iyz="-0.000291" izz="0.023619"/>
+  </inertial>
+  <visual>
+    <origin rpy="0 0 0" xyz="0.0 -0.05 -0.18"/>
+    <geometry>
+      <mesh filename="package://arm_export_description/meshes/base_turnable_v14_1.stl" scale="0.001 0.001 0.001"/>
+    </geometry>
+    <material name="silver"/>
+  </visual>
+  <collision>
+    <origin rpy="0 0 0" xyz="0.0 -0.05 -0.18"/>
+    <geometry>
+      <mesh filename="package://arm_export_description/meshes/base_turnable_v14_1.stl" scale="0.001 0.001 0.001"/>
+    </geometry>
+  </collision>
+</link>
 <link name="NEMA_34_v2_1">
   <inertial>
-    <origin rpy="0 0 0" xyz="-3.2210029226501892e-06 0.0 0.07651505285685495"/>
-    <mass value="5.316520087759884"/>
-    <inertia ixx="0.014133" ixy="-0.0" ixz="-2e-06" iyy="0.014133" iyz="0.0" izz="0.005731"/>
-  </inertial>
-  <visual>
-    <origin rpy="0 0 0" xyz="0.0 0.075 -0.06"/>
-    <geometry>
-      <mesh filename="package://arm_export_description/meshes/NEMA_34_v2_1.stl" scale="0.001 0.001 0.001"/>
-    </geometry>
-    <material name="silver"/>
-  </visual>
-  <collision>
-    <origin rpy="0 0 0" xyz="0.0 0.075 -0.06"/>
-    <geometry>
-      <mesh filename="package://arm_export_description/meshes/NEMA_34_v2_1.stl" scale="0.001 0.001 0.001"/>
-    </geometry>
-  </collision>
-</link>
-<link name="base_turnable_v8_1">
-  <inertial>
-    <origin rpy="0 0 0" xyz="-0.001007798204056028 0.008254459699838873 -0.040805505989257335"/>
-    <mass value="4.032845174316641"/>
-    <inertia ixx="0.020961" ixy="0.000332" ixz="0.000389" iyy="0.018599" iyz="-0.003189" izz="0.008486"/>
-  </inertial>
-  <visual>
-    <origin rpy="0 0 0" xyz="-0.0 -0.06 -0.16"/>
-    <geometry>
-      <mesh filename="package://arm_export_description/meshes/base_turnable_v8_1.stl" scale="0.001 0.001 0.001"/>
-    </geometry>
-    <material name="silver"/>
-  </visual>
-  <collision>
-    <origin rpy="0 0 0" xyz="-0.0 -0.06 -0.16"/>
-    <geometry>
-      <mesh filename="package://arm_export_description/meshes/base_turnable_v8_1.stl" scale="0.001 0.001 0.001"/>
-    </geometry>
-  </collision>
-</link>
-<link name="NEMA_34_v2__1__1">
-  <inertial>
-    <origin rpy="0 0 0" xyz="0.07651505285685478 -5.551115123125783e-17 3.2210029226598103e-06"/>
+    <origin rpy="0 0 0" xyz="0.07651505285685478 -5.551115123125783e-17 3.221002922604299e-06"/>
     <mass value="5.316520087759884"/>
     <inertia ixx="0.005731" ixy="0.0" ixz="2e-06" iyy="0.014133" iyz="0.0" izz="0.014133"/>
   </inertial>
   <visual>
-    <origin rpy="0 0 0" xyz="-0.04 -0.15 -0.215"/>
-    <geometry>
-      <mesh filename="package://arm_export_description/meshes/NEMA_34_v2__1__1.stl" scale="0.001 0.001 0.001"/>
-    </geometry>
-    <material name="silver"/>
-  </visual>
-  <collision>
-    <origin rpy="0 0 0" xyz="-0.04 -0.15 -0.215"/>
-    <geometry>
-      <mesh filename="package://arm_export_description/meshes/NEMA_34_v2__1__1.stl" scale="0.001 0.001 0.001"/>
-    </geometry>
-  </collision>
-</link>
-<link name="stepper_joint_v6__1__1">
-  <inertial>
-    <origin rpy="0 0 0" xyz="0.0075000000000001316 2.7755575615628914e-17 -1.3053447212030278e-13"/>
+    <origin rpy="0 0 0" xyz="-0.04 -0.14 -0.265"/>
+    <geometry>
+      <mesh filename="package://arm_export_description/meshes/NEMA_34_v2_1.stl" scale="0.001 0.001 0.001"/>
+    </geometry>
+    <material name="silver"/>
+  </visual>
+  <collision>
+    <origin rpy="0 0 0" xyz="-0.04 -0.14 -0.265"/>
+    <geometry>
+      <mesh filename="package://arm_export_description/meshes/NEMA_34_v2_1.stl" scale="0.001 0.001 0.001"/>
+    </geometry>
+  </collision>
+</link>
+<link name="stepper_joint_v6_1">
+  <inertial>
+    <origin rpy="0 0 0" xyz="0.0075000000000001316 0.0 -1.305622276959184e-13"/>
     <mass value="0.03498948817935604"/>
-    <inertia ixx="7e-06" ixy="0.0" ixz="0.0" iyy="4e-06" iyz="0.0" izz="4e-06"/>
-  </inertial>
-  <visual>
-    <origin rpy="0 0 0" xyz="-0.00348 -0.15 -0.215"/>
-    <geometry>
-      <mesh filename="package://arm_export_description/meshes/stepper_joint_v6__1__1.stl" scale="0.001 0.001 0.001"/>
-    </geometry>
-    <material name="silver"/>
-  </visual>
-  <collision>
-    <origin rpy="0 0 0" xyz="-0.00348 -0.15 -0.215"/>
-    <geometry>
-      <mesh filename="package://arm_export_description/meshes/stepper_joint_v6__1__1.stl" scale="0.001 0.001 0.001"/>
-    </geometry>
-  </collision>
-</link>
-<link name="stepper_joint_v6_1">
-  <inertial>
-    <origin rpy="0 0 0" xyz="1.3042541342589262e-13 5.551115123125783e-17 0.007500000000000059"/>
-    <mass value="0.03498948817935604"/>
-    <inertia ixx="4e-06" ixy="0.0" ixz="-0.0" iyy="4e-06" iyz="0.0" izz="7e-06"/>
-  </inertial>
-  <visual>
-    <origin rpy="0 0 0" xyz="0.0 0.075 -0.02348"/>
+    <inertia ixx="7e-06" ixy="0.0" ixz="-0.0" iyy="4e-06" iyz="0.0" izz="4e-06"/>
+  </inertial>
+  <visual>
+    <origin rpy="0 0 0" xyz="-0.00348 -0.14 -0.265"/>
     <geometry>
       <mesh filename="package://arm_export_description/meshes/stepper_joint_v6_1.stl" scale="0.001 0.001 0.001"/>
@@ -118,5 +78,5 @@
   </visual>
   <collision>
-    <origin rpy="0 0 0" xyz="0.0 0.075 -0.02348"/>
+    <origin rpy="0 0 0" xyz="-0.00348 -0.14 -0.265"/>
     <geometry>
       <mesh filename="package://arm_export_description/meshes/stepper_joint_v6_1.stl" scale="0.001 0.001 0.001"/>
@@ -126,10 +86,10 @@
 <link name="link_1_v13_1">
   <inertial>
-    <origin rpy="0 0 0" xyz="-0.007499999999999868 0.2614820661654451 -2.7755575615628914e-17"/>
+    <origin rpy="0 0 0" xyz="-0.007499999999999868 0.2614820661654451 0.0"/>
     <mass value="1.2422891158221263"/>
-    <inertia ixx="0.03033" ixy="0.0" ixz="-0.0" iyy="0.000414" iyz="-0.0" izz="0.029962"/>
-  </inertial>
-  <visual>
-    <origin rpy="0 0 0" xyz="-0.00348 -0.15 -0.215"/>
+    <inertia ixx="0.03033" ixy="0.0" ixz="-0.0" iyy="0.000414" iyz="0.0" izz="0.029962"/>
+  </inertial>
+  <visual>
+    <origin rpy="0 0 0" xyz="-0.00348 -0.14 -0.265"/>
     <geometry>
       <mesh filename="package://arm_export_description/meshes/link_1_v13_1.stl" scale="0.001 0.001 0.001"/>
@@ -138,5 +98,5 @@
   </visual>
   <collision>
-    <origin rpy="0 0 0" xyz="-0.00348 -0.15 -0.215"/>
+    <origin rpy="0 0 0" xyz="-0.00348 -0.14 -0.265"/>
     <geometry>
       <mesh filename="package://arm_export_description/meshes/link_1_v13_1.stl" scale="0.001 0.001 0.001"/>
@@ -146,10 +106,10 @@
 <link name="link_2_v8_1">
   <inertial>
-    <origin rpy="0 0 0" xyz="0.02499852381758487 0.17692221361514127 2.7755575615628914e-17"/>
+    <origin rpy="0 0 0" xyz="0.02499852381758487 0.1769222136151415 0.0"/>
     <mass value="1.5478777520934175"/>
     <inertia ixx="0.032303" ixy="-0.002603" ixz="-0.0" iyy="0.001209" iyz="-0.0" izz="0.032482"/>
   </inertial>
   <visual>
-    <origin rpy="0 0 0" xyz="-0.03848 -0.735 -0.215"/>
+    <origin rpy="0 0 0" xyz="-0.03848 -0.725 -0.265"/>
     <geometry>
       <mesh filename="package://arm_export_description/meshes/link_2_v8_1.stl" scale="0.001 0.001 0.001"/>
@@ -158,5 +118,5 @@
   </visual>
   <collision>
-    <origin rpy="0 0 0" xyz="-0.03848 -0.735 -0.215"/>
+    <origin rpy="0 0 0" xyz="-0.03848 -0.725 -0.265"/>
     <geometry>
       <mesh filename="package://arm_export_description/meshes/link_2_v8_1.stl" scale="0.001 0.001 0.001"/>
@@ -171,5 +131,5 @@
   </inertial>
   <visual>
-    <origin rpy="0 0 0" xyz="-0.06848 -1.19 -0.215"/>
+    <origin rpy="0 0 0" xyz="-0.06848 -1.18 -0.265"/>
     <geometry>
       <mesh filename="package://arm_export_description/meshes/joint_end_v3_1.stl" scale="0.001 0.001 0.001"/>
@@ -178,5 +138,5 @@
   </visual>
   <collision>
-    <origin rpy="0 0 0" xyz="-0.06848 -1.19 -0.215"/>
+    <origin rpy="0 0 0" xyz="-0.06848 -1.18 -0.265"/>
     <geometry>
       <mesh filename="package://arm_export_description/meshes/joint_end_v3_1.stl" scale="0.001 0.001 0.001"/>
@@ -184,41 +144,41 @@
   </collision>
 </link>
-<link name="NEMA_24_v1__2__1">
-  <inertial>
-    <origin rpy="0 0 0" xyz="0.04795079485405239 7.655954098462203e-08 2.5568133203979215e-06"/>
+<link name="NEMA_24_v1__1__1">
+  <inertial>
+    <origin rpy="0 0 0" xyz="0.04795079485405239 7.655954092911088e-08 2.5568133203979215e-06"/>
     <mass value="2.4982959259379585"/>
     <inertia ixx="0.001293" ixy="-0.0" ixz="-0.0" iyy="0.002718" iyz="0.0" izz="0.002718"/>
   </inertial>
   <visual>
-    <origin rpy="0 0 0" xyz="-0.00348 -0.2875 -0.215"/>
-    <geometry>
-      <mesh filename="package://arm_export_description/meshes/NEMA_24_v1__2__1.stl" scale="0.001 0.001 0.001"/>
-    </geometry>
-    <material name="silver"/>
-  </visual>
-  <collision>
-    <origin rpy="0 0 0" xyz="-0.00348 -0.2875 -0.215"/>
-    <geometry>
-      <mesh filename="package://arm_export_description/meshes/NEMA_24_v1__2__1.stl" scale="0.001 0.001 0.001"/>
-    </geometry>
-  </collision>
-</link>
-<link name="NEMA_24_v1_1">
-  <inertial>
-    <origin rpy="0 0 0" xyz="7.65595409013553e-08 -0.04795079485405229 2.556813320425677e-06"/>
+    <origin rpy="0 0 0" xyz="-0.00348 -0.2775 -0.265"/>
+    <geometry>
+      <mesh filename="package://arm_export_description/meshes/NEMA_24_v1__1__1.stl" scale="0.001 0.001 0.001"/>
+    </geometry>
+    <material name="silver"/>
+  </visual>
+  <collision>
+    <origin rpy="0 0 0" xyz="-0.00348 -0.2775 -0.265"/>
+    <geometry>
+      <mesh filename="package://arm_export_description/meshes/NEMA_24_v1__1__1.stl" scale="0.001 0.001 0.001"/>
+    </geometry>
+  </collision>
+</link>
+<link name="NEMA_24_v1__3__1">
+  <inertial>
+    <origin rpy="0 0 0" xyz="7.65595409013553e-08 -0.04795079485405218 2.5568133203979215e-06"/>
     <mass value="2.4982959259379585"/>
     <inertia ixx="0.002718" ixy="0.0" ixz="0.0" iyy="0.001293" iyz="0.0" izz="0.002718"/>
   </inertial>
   <visual>
-    <origin rpy="0 0 0" xyz="-0.03848 -0.635 -0.215"/>
-    <geometry>
-      <mesh filename="package://arm_export_description/meshes/NEMA_24_v1_1.stl" scale="0.001 0.001 0.001"/>
-    </geometry>
-    <material name="silver"/>
-  </visual>
-  <collision>
-    <origin rpy="0 0 0" xyz="-0.03848 -0.635 -0.215"/>
-    <geometry>
-      <mesh filename="package://arm_export_description/meshes/NEMA_24_v1_1.stl" scale="0.001 0.001 0.001"/>
+    <origin rpy="0 0 0" xyz="-0.03848 -0.625 -0.265"/>
+    <geometry>
+      <mesh filename="package://arm_export_description/meshes/NEMA_24_v1__3__1.stl" scale="0.001 0.001 0.001"/>
+    </geometry>
+    <material name="silver"/>
+  </visual>
+  <collision>
+    <origin rpy="0 0 0" xyz="-0.03848 -0.625 -0.265"/>
+    <geometry>
+      <mesh filename="package://arm_export_description/meshes/NEMA_24_v1__3__1.stl" scale="0.001 0.001 0.001"/>
     </geometry>
   </collision>
@@ -228,8 +188,8 @@
     <origin rpy="0 0 0" xyz="0.026213672668365277 0.017799785433927795 0.0"/>
     <mass value="0.8743627585315773"/>
-    <inertia ixx="0.000992" ixy="-8.4e-05" ixz="0.0" iyy="0.000864" iyz="0.0" izz="0.001253"/>
-  </inertial>
-  <visual>
-    <origin rpy="0 0 0" xyz="-0.00348 -0.665 -0.215"/>
+    <inertia ixx="0.000992" ixy="-8.4e-05" ixz="0.0" iyy="0.000864" iyz="-0.0" izz="0.001253"/>
+  </inertial>
+  <visual>
+    <origin rpy="0 0 0" xyz="-0.00348 -0.655 -0.265"/>
     <geometry>
       <mesh filename="package://arm_export_description/meshes/joint_v6_1.stl" scale="0.001 0.001 0.001"/>
@@ -238,5 +198,5 @@
   </visual>
   <collision>
-    <origin rpy="0 0 0" xyz="-0.00348 -0.665 -0.215"/>
+    <origin rpy="0 0 0" xyz="-0.00348 -0.655 -0.265"/>
     <geometry>
       <mesh filename="package://arm_export_description/meshes/joint_v6_1.stl" scale="0.001 0.001 0.001"/>
@@ -244,47 +204,157 @@
   </collision>
 </link>
-<link name="NEMA_24_v1__1__1">
-  <inertial>
-    <origin rpy="0 0 0" xyz="-7.655954063073844e-08 -0.047450794854052236 -0.03000255681332048"/>
+<link name="NEMA_24_v1__2__1">
+  <inertial>
+    <origin rpy="0 0 0" xyz="7.655954077029509e-08 2.5568133205228216e-06 0.047950794854052264"/>
+    <mass value="2.4982959259379585"/>
+    <inertia ixx="0.002718" ixy="0.0" ixz="-0.0" iyy="0.002718" iyz="-0.0" izz="0.001293"/>
+  </inertial>
+  <visual>
+    <origin rpy="0 0 0" xyz="0.0 0.075 -0.06"/>
+    <geometry>
+      <mesh filename="package://arm_export_description/meshes/NEMA_24_v1__2__1.stl" scale="0.001 0.001 0.001"/>
+    </geometry>
+    <material name="silver"/>
+  </visual>
+  <collision>
+    <origin rpy="0 0 0" xyz="0.0 0.075 -0.06"/>
+    <geometry>
+      <mesh filename="package://arm_export_description/meshes/NEMA_24_v1__2__1.stl" scale="0.001 0.001 0.001"/>
+    </geometry>
+  </collision>
+</link>
+<link name="Intel_RealSense_D435_v3_1">
+  <inertial>
+    <origin rpy="0 0 0" xyz="-0.0010696020063957895 0.0010440004277678036 0.012511380076091427"/>
+    <mass value="0.2739287989936542"/>
+    <inertia ixx="2.6e-05" ixy="-2e-06" ixz="0.0" iyy="0.000177" iyz="0.0" izz="0.000178"/>
+  </inertial>
+  <visual>
+    <origin rpy="0 0 0" xyz="0.09 -0.055 -1.209827"/>
+    <geometry>
+      <mesh filename="package://arm_export_description/meshes/Intel_RealSense_D435_v3_1.stl" scale="0.001 0.001 0.001"/>
+    </geometry>
+    <material name="silver"/>
+  </visual>
+  <collision>
+    <origin rpy="0 0 0" xyz="0.09 -0.055 -1.209827"/>
+    <geometry>
+      <mesh filename="package://arm_export_description/meshes/Intel_RealSense_D435_v3_1.stl" scale="0.001 0.001 0.001"/>
+    </geometry>
+  </collision>
+</link>
+<link name="NEMA_24_v1_1">
+  <inertial>
+    <origin rpy="0 0 0" xyz="-7.655954063073844e-08 0.0009492051459477624 -0.02980255681332042"/>
     <mass value="2.4982959259379585"/>
     <inertia ixx="0.002718" ixy="-0.0" ixz="0.0" iyy="0.001293" iyz="-0.0" izz="0.002718"/>
   </inertial>
   <visual>
-    <origin rpy="0 0 0" xyz="-0.03598 -0.735 -0.185"/>
-    <geometry>
-      <mesh filename="package://arm_export_description/meshes/NEMA_24_v1__1__1.stl" scale="0.001 0.001 0.001"/>
-    </geometry>
-    <material name="silver"/>
-  </visual>
-  <collision>
-    <origin rpy="0 0 0" xyz="-0.03598 -0.735 -0.185"/>
-    <geometry>
-      <mesh filename="package://arm_export_description/meshes/NEMA_24_v1__1__1.stl" scale="0.001 0.001 0.001"/>
-    </geometry>
-  </collision>
-</link>
-<joint name="Rigid15" type="fixed">
-  <origin rpy="0 0 0" xyz="0.0 -0.075 0.06"/>
+    <origin rpy="0 0 0" xyz="-0.03598 -0.675 -0.235"/>
+    <geometry>
+      <mesh filename="package://arm_export_description/meshes/NEMA_24_v1_1.stl" scale="0.001 0.001 0.001"/>
+    </geometry>
+    <material name="silver"/>
+  </visual>
+  <collision>
+    <origin rpy="0 0 0" xyz="-0.03598 -0.675 -0.235"/>
+    <geometry>
+      <mesh filename="package://arm_export_description/meshes/NEMA_24_v1_1.stl" scale="0.001 0.001 0.001"/>
+    </geometry>
+  </collision>
+</link>
+<link name="gripper_export_v2_1">
+  <inertial>
+    <origin rpy="0 0 0" xyz="-8.738046813894229e-10 0.03673655788581853 1.1906842178888155e-10"/>
+    <mass value="1.1315792783817065"/>
+    <inertia ixx="0.001126" ixy="0.0" ixz="-0.0" iyy="0.001318" iyz="-0.0" izz="0.001126"/>
+  </inertial>
+  <visual>
+    <origin rpy="0 0 0" xyz="-0.02848 -1.23 -0.265"/>
+    <geometry>
+      <mesh filename="package://arm_export_description/meshes/gripper_export_v2_1.stl" scale="0.001 0.001 0.001"/>
+    </geometry>
+    <material name="silver"/>
+  </visual>
+  <collision>
+    <origin rpy="0 0 0" xyz="-0.02848 -1.23 -0.265"/>
+    <geometry>
+      <mesh filename="package://arm_export_description/meshes/gripper_export_v2_1.stl" scale="0.001 0.001 0.001"/>
+    </geometry>
+  </collision>
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