Commit message: robot joints renamed

File: fusion_360_export/Robot_description/urdf/Robot.xacro (robot description, xacro)
@@ -1,17 +1,17 @@
 <?xml version="1.0" ?>
-<robot name="Robot" xmlns:xacro="http://www.ros.org/wiki/xacro">
-<xacro:include filename="$(find Robot_description)/urdf/materials.xacro" />
-<xacro:include filename="$(find Robot_description)/urdf/Robot.trans" />
-<xacro:include filename="$(find Robot_description)/urdf/Robot.gazebo" />
+<robot name="robot" xmlns:xacro="http://www.ros.org/wiki/xacro">
+<xacro:include filename="$(find robot_description)/urdf/materials.xacro" />
+<xacro:include filename="$(find robot_description)/urdf/robot.trans" />
+<xacro:include filename="$(find robot_description)/urdf/robot.gazebo" />
 <link name="base_link">
   <inertial>
-    <origin rpy="0 0 0" xyz="0.004639774814419823 1.4771468453425644e-05 0.22530002486564402"/>
+    <origin rpy="0 0 0" xyz="-1.4771468453599796e-05 -0.4394102251855798 -0.5105474620020639"/>
     <mass value="90.2870635836035"/>
-    <inertia ixx="10.456164" ixy="1.4e-05" ixz="-0.360506" iyy="16.958749" iyz="0.000256" izz="18.430844"/>
+    <inertia ixx="16.958749" ixy="-1.4e-05" ixz="-0.000256" iyy="10.456164" iyz="-0.360506" izz="18.430844"/>
   </inertial>
   <visual>
     <origin rpy="0 0 0" xyz="0 0 0"/>
     <geometry>
-      <mesh filename="package://Robot_description/meshes/base_link.stl" scale="0.001 0.001 0.001"/>
+      <mesh filename="package://robot_description/meshes/base_link.stl" scale="0.001 0.001 0.001"/>
     </geometry>
     <material name="silver"/>
@@ -20,5 +20,5 @@
     <origin rpy="0 0 0" xyz="0 0 0"/>
     <geometry>
-      <mesh filename="package://Robot_description/meshes/base_link.stl" scale="0.001 0.001 0.001"/>
+      <mesh filename="package://robot_description/meshes/base_link.stl" scale="0.001 0.001 0.001"/>
     </geometry>
   </collision>
@@ -26,538 +26,564 @@
 <link name="arm_base_1">
   <inertial>
-    <origin rpy="0 0 0" xyz="-0.10852318160677482 9.021804964276997e-14 0.07021798038523674"/>
+    <origin rpy="0 0 0" xyz="-9.028631835610602e-14 -0.10852318160677443 0.07021749351752887"/>
     <mass value="2.9829690964186772"/>
-    <inertia ixx="0.017973" ixy="0.0" ixz="-0.002884" iyy="0.024074" iyz="0.0" izz="0.02919"/>
-  </inertial>
-  <visual>
-    <origin rpy="0 0 0" xyz="-0.51905 -0.0 -0.555847"/>
-    <geometry>
-      <mesh filename="package://Robot_description/meshes/arm_base_1.stl" scale="0.001 0.001 0.001"/>
-    </geometry>
-    <material name="silver"/>
-  </visual>
-  <collision>
-    <origin rpy="0 0 0" xyz="-0.51905 -0.0 -0.555847"/>
-    <geometry>
-      <mesh filename="package://Robot_description/meshes/arm_base_1.stl" scale="0.001 0.001 0.001"/>
-    </geometry>
-  </collision>
-</link>
-<link name="base_turnable_v14_1">
-  <inertial>
-    <origin rpy="0 0 0" xyz="0.004673714897230008 0.029934483757072104 0.10053910370878505"/>
-    <mass value="7.350921302447738"/>
-    <inertia ixx="0.40707" ixy="0.000566" ixz="-0.000291" iyy="0.39669" iyz="-0.055433" izz="0.023619"/>
-  </inertial>
-  <visual>
-    <origin rpy="0 0 0" xyz="-0.44405 0.0 -0.735847"/>
-    <geometry>
-      <mesh filename="package://Robot_description/meshes/base_turnable_v14_1.stl" scale="0.001 0.001 0.001"/>
-    </geometry>
-    <material name="silver"/>
-  </visual>
-  <collision>
-    <origin rpy="0 0 0" xyz="-0.44405 0.0 -0.735847"/>
-    <geometry>
-      <mesh filename="package://Robot_description/meshes/base_turnable_v14_1.stl" scale="0.001 0.001 0.001"/>
-    </geometry>
-  </collision>
-</link>
-<link name="NEMA_34_v2_1">
-  <inertial>
-    <origin rpy="0 0 0" xyz="-3.221002877085155e-06 -0.07651505285685486 4.86867707816252e-07"/>
-    <mass value="5.3165200877598835"/>
-    <inertia ixx="0.014133" ixy="2e-06" ixz="0.0" iyy="0.005731" iyz="0.0" izz="0.014133"/>
-  </inertial>
-  <visual>
-    <origin rpy="0 0 0" xyz="-0.53405 0.04 -0.820847"/>
-    <geometry>
-      <mesh filename="package://Robot_description/meshes/NEMA_34_v2_1.stl" scale="0.001 0.001 0.001"/>
-    </geometry>
-    <material name="silver"/>
-  </visual>
-  <collision>
-    <origin rpy="0 0 0" xyz="-0.53405 0.04 -0.820847"/>
-    <geometry>
-      <mesh filename="package://Robot_description/meshes/NEMA_34_v2_1.stl" scale="0.001 0.001 0.001"/>
-    </geometry>
-  </collision>
-</link>
-<link name="stepper_joint_v6_1">
-  <inertial>
-    <origin rpy="0 0 0" xyz="1.3000711618360583e-13 -0.0075000000000001316 4.86867707816252e-07"/>
+    <inertia ixx="0.024074" ixy="-0.0" ixz="-0.0" iyy="0.017973" iyz="-0.002884" izz="0.02919"/>
+  </inertial>
+  <visual>
+    <origin rpy="0 0 0" xyz="0.0 -0.075 0.18"/>
+    <geometry>
+      <mesh filename="package://robot_description/meshes/arm_base_1.stl" scale="0.001 0.001 0.001"/>
+    </geometry>
+    <material name="silver"/>
+  </visual>
+  <collision>
+    <origin rpy="0 0 0" xyz="0.0 -0.075 0.18"/>
+    <geometry>
+      <mesh filename="package://robot_description/meshes/arm_base_1.stl" scale="0.001 0.001 0.001"/>
+    </geometry>
+  </collision>
+</link>
+<link name="stepper_joint_1">
+  <inertial>
+    <origin rpy="0 0 0" xyz="0.007499999999999989 1.3028467193976212e-13 1.3877787807814457e-16"/>
     <mass value="0.03498948817935604"/>
-    <inertia ixx="4e-06" ixy="-0.0" ixz="0.0" iyy="7e-06" iyz="-0.0" izz="4e-06"/>
-  </inertial>
-  <visual>
-    <origin rpy="0 0 0" xyz="-0.53405 0.00348 -0.820847"/>
-    <geometry>
-      <mesh filename="package://Robot_description/meshes/stepper_joint_v6_1.stl" scale="0.001 0.001 0.001"/>
-    </geometry>
-    <material name="silver"/>
-  </visual>
-  <collision>
-    <origin rpy="0 0 0" xyz="-0.53405 0.00348 -0.820847"/>
-    <geometry>
-      <mesh filename="package://Robot_description/meshes/stepper_joint_v6_1.stl" scale="0.001 0.001 0.001"/>
-    </geometry>
-  </collision>
-</link>
-<link name="link_1_v13_1">
-  <inertial>
-    <origin rpy="0 0 0" xyz="0.2614820661654448 0.00749999999999987 4.86867707816252e-07"/>
+    <inertia ixx="7e-06" ixy="0.0" ixz="0.0" iyy="4e-06" iyz="0.0" izz="4e-06"/>
+  </inertial>
+  <visual>
+    <origin rpy="0 0 0" xyz="-0.00348 -0.09 -0.085"/>
+    <geometry>
+      <mesh filename="package://robot_description/meshes/stepper_joint_1.stl" scale="0.001 0.001 0.001"/>
+    </geometry>
+    <material name="silver"/>
+  </visual>
+  <collision>
+    <origin rpy="0 0 0" xyz="-0.00348 -0.09 -0.085"/>
+    <geometry>
+      <mesh filename="package://robot_description/meshes/stepper_joint_1.stl" scale="0.001 0.001 0.001"/>
+    </geometry>
+  </collision>
+</link>
+<link name="link_1_1">
+  <inertial>
+    <origin rpy="0 0 0" xyz="-0.00750000000000001 0.2614820661654451 1.3877787807814457e-16"/>
     <mass value="1.2422891158221263"/>
-    <inertia ixx="0.000414" ixy="-0.0" ixz="-0.0" iyy="0.03033" iyz="0.0" izz="0.029962"/>
-  </inertial>
-  <visual>
-    <origin rpy="0 0 0" xyz="-0.53405 0.00348 -0.820847"/>
-    <geometry>
-      <mesh filename="package://Robot_description/meshes/link_1_v13_1.stl" scale="0.001 0.001 0.001"/>
-    </geometry>
-    <material name="silver"/>
-  </visual>
-  <collision>
-    <origin rpy="0 0 0" xyz="-0.53405 0.00348 -0.820847"/>
-    <geometry>
-      <mesh filename="package://Robot_description/meshes/link_1_v13_1.stl" scale="0.001 0.001 0.001"/>
-    </geometry>
-  </collision>
-</link>
-<link name="joint_v6_1">
-  <inertial>
-    <origin rpy="0 0 0" xyz="0.01779978543392735 -0.026213672668365277 4.86867707816252e-07"/>
+    <inertia ixx="0.03033" ixy="0.0" ixz="0.0" iyy="0.000414" iyz="-0.0" izz="0.029962"/>
+  </inertial>
+  <visual>
+    <origin rpy="0 0 0" xyz="-0.00348 -0.09 -0.085"/>
+    <geometry>
+      <mesh filename="package://robot_description/meshes/link_1_1.stl" scale="0.001 0.001 0.001"/>
+    </geometry>
+    <material name="silver"/>
+  </visual>
+  <collision>
+    <origin rpy="0 0 0" xyz="-0.00348 -0.09 -0.085"/>
+    <geometry>
+      <mesh filename="package://robot_description/meshes/link_1_1.stl" scale="0.001 0.001 0.001"/>
+    </geometry>
+  </collision>
+</link>
+<link name="link_2_1">
+  <inertial>
+    <origin rpy="0 0 0" xyz="0.026213672668365277 0.017799785433927795 1.3877787807814457e-16"/>
     <mass value="0.8743627585315773"/>
-    <inertia ixx="0.000864" ixy="8.4e-05" ixz="0.0" iyy="0.000992" iyz="0.0" izz="0.001253"/>
-  </inertial>
-  <visual>
-    <origin rpy="0 0 0" xyz="-1.04905 0.00348 -0.820847"/>
-    <geometry>
-      <mesh filename="package://Robot_description/meshes/joint_v6_1.stl" scale="0.001 0.001 0.001"/>
-    </geometry>
-    <material name="silver"/>
-  </visual>
-  <collision>
-    <origin rpy="0 0 0" xyz="-1.04905 0.00348 -0.820847"/>
-    <geometry>
-      <mesh filename="package://Robot_description/meshes/joint_v6_1.stl" scale="0.001 0.001 0.001"/>
-    </geometry>
-  </collision>
-</link>
-<link name="link_2_v8_1">
-  <inertial>
-    <origin rpy="0 0 0" xyz="0.17692221361514116 -0.02499852381758487 4.868677079272743e-07"/>
+    <inertia ixx="0.000992" ixy="-8.4e-05" ixz="0.0" iyy="0.000864" iyz="0.0" izz="0.001253"/>
+  </inertial>
+  <visual>
+    <origin rpy="0 0 0" xyz="-0.00348 -0.605 -0.085"/>
+    <geometry>
+      <mesh filename="package://robot_description/meshes/link_2_1.stl" scale="0.001 0.001 0.001"/>
+    </geometry>
+    <material name="silver"/>
+  </visual>
+  <collision>
+    <origin rpy="0 0 0" xyz="-0.00348 -0.605 -0.085"/>
+    <geometry>
+      <mesh filename="package://robot_description/meshes/link_2_1.stl" scale="0.001 0.001 0.001"/>
+    </geometry>
+  </collision>
+</link>
+<link name="link_3_1">
+  <inertial>
+    <origin rpy="0 0 0" xyz="0.02499852381758487 0.1769222136151417 3.885780586188048e-16"/>
     <mass value="1.5478777520934175"/>
-    <inertia ixx="0.001209" ixy="0.002603" ixz="-0.0" iyy="0.032303" iyz="0.0" izz="0.032482"/>
-  </inertial>
-  <visual>
-    <origin rpy="0 0 0" xyz="-1.11905 0.03848 -0.820847"/>
-    <geometry>
-      <mesh filename="package://Robot_description/meshes/link_2_v8_1.stl" scale="0.001 0.001 0.001"/>
-    </geometry>
-    <material name="silver"/>
-  </visual>
-  <collision>
-    <origin rpy="0 0 0" xyz="-1.11905 0.03848 -0.820847"/>
-    <geometry>
-      <mesh filename="package://Robot_description/meshes/link_2_v8_1.stl" scale="0.001 0.001 0.001"/>
-    </geometry>
-  </collision>
-</link>
-<link name="joint_end_v3_1">
-  <inertial>
-    <origin rpy="0 0 0" xyz="0.011579118062804206 0.03379678599677132 4.868677079272743e-07"/>
+    <inertia ixx="0.032303" ixy="-0.002603" ixz="0.0" iyy="0.001209" iyz="0.0" izz="0.032482"/>
+  </inertial>
+  <visual>
+    <origin rpy="0 0 0" xyz="-0.03848 -0.675 -0.085"/>
+    <geometry>
+      <mesh filename="package://robot_description/meshes/link_3_1.stl" scale="0.001 0.001 0.001"/>
+    </geometry>
+    <material name="silver"/>
+  </visual>
+  <collision>
+    <origin rpy="0 0 0" xyz="-0.03848 -0.675 -0.085"/>
+    <geometry>
+      <mesh filename="package://robot_description/meshes/link_3_1.stl" scale="0.001 0.001 0.001"/>
+    </geometry>
+  </collision>
+</link>
+<link name="link_end_1">
+  <inertial>
+    <origin rpy="0 0 0" xyz="-0.03379678599677132 0.011579118062804872 4.163336342344337e-16"/>
     <mass value="1.063293416063342"/>
-    <inertia ixx="0.00115" ixy="-7.6e-05" ixz="-0.0" iyy="0.000747" iyz="-0.0" izz="0.001353"/>
-  </inertial>
-  <visual>
-    <origin rpy="0 0 0" xyz="-1.57405 0.06848 -0.820847"/>
-    <geometry>
-      <mesh filename="package://Robot_description/meshes/joint_end_v3_1.stl" scale="0.001 0.001 0.001"/>
-    </geometry>
-    <material name="silver"/>
-  </visual>
-  <collision>
-    <origin rpy="0 0 0" xyz="-1.57405 0.06848 -0.820847"/>
-    <geometry>
-      <mesh filename="package://Robot_description/meshes/joint_end_v3_1.stl" scale="0.001 0.001 0.001"/>
-    </geometry>
-  </collision>
-</link>
-<link name="NEMA_24_v1_1">
-  <inertial>
-    <origin rpy="0 0 0" xyz="7.655954076257743e-08 2.556813320462289e-06 0.04795128172176"/>
+    <inertia ixx="0.000747" ixy="7.6e-05" ixz="0.0" iyy="0.00115" iyz="-0.0" izz="0.001353"/>
+  </inertial>
+  <visual>
+    <origin rpy="0 0 0" xyz="-0.06848 -1.13 -0.085"/>
+    <geometry>
+      <mesh filename="package://robot_description/meshes/link_end_1.stl" scale="0.001 0.001 0.001"/>
+    </geometry>
+    <material name="silver"/>
+  </visual>
+  <collision>
+    <origin rpy="0 0 0" xyz="-0.06848 -1.13 -0.085"/>
+    <geometry>
+      <mesh filename="package://robot_description/meshes/link_end_1.stl" scale="0.001 0.001 0.001"/>
+    </geometry>
+  </collision>
+</link>
+<link name="NEMA_24_1_1">
+  <inertial>
+    <origin rpy="0 0 0" xyz="-2.5568133205304072e-06 7.655954109564433e-08 0.047950794854052264"/>
     <mass value="2.4982959259379585"/>
-    <inertia ixx="0.002718" ixy="0.0" ixz="-0.0" iyy="0.002718" iyz="-0.0" izz="0.001293"/>
-  </inertial>
-  <visual>
-    <origin rpy="0 0 0" xyz="-0.31905 0.0 -0.615847"/>
-    <geometry>
-      <mesh filename="package://Robot_description/meshes/NEMA_24_v1_1.stl" scale="0.001 0.001 0.001"/>
-    </geometry>
-    <material name="silver"/>
-  </visual>
-  <collision>
-    <origin rpy="0 0 0" xyz="-0.31905 0.0 -0.615847"/>
-    <geometry>
-      <mesh filename="package://Robot_description/meshes/NEMA_24_v1_1.stl" scale="0.001 0.001 0.001"/>
-    </geometry>
-  </collision>
-</link>
-<link name="NEMA_24_v1__1__1">
-  <inertial>
-    <origin rpy="0 0 0" xyz="7.655954081808858e-08 -0.047950794854052424 3.0436810282141735e-06"/>
+    <inertia ixx="0.002718" ixy="-0.0" ixz="0.0" iyy="0.002718" iyz="-0.0" izz="0.001293"/>
+  </inertial>
+  <visual>
+    <origin rpy="0 0 0" xyz="-0.0 0.125 0.12"/>
+    <geometry>
+      <mesh filename="package://robot_description/meshes/NEMA_24_1_1.stl" scale="0.001 0.001 0.001"/>
+    </geometry>
+    <material name="silver"/>
+  </visual>
+  <collision>
+    <origin rpy="0 0 0" xyz="-0.0 0.125 0.12"/>
+    <geometry>
+      <mesh filename="package://robot_description/meshes/NEMA_24_1_1.stl" scale="0.001 0.001 0.001"/>
+    </geometry>
+  </collision>
+</link>
+<link name="NEMA_24_2_1">
+  <inertial>
+    <origin rpy="0 0 0" xyz="0.04795079485405226 7.655954106788876e-08 2.556813320619966e-06"/>
+    <mass value="2.4982959259379585"/>
+    <inertia ixx="0.001293" ixy="-0.0" ixz="-0.0" iyy="0.002718" iyz="0.0" izz="0.002718"/>
+  </inertial>
+  <visual>
+    <origin rpy="0 0 0" xyz="-0.00348 -0.2275 -0.085"/>
+    <geometry>
+      <mesh filename="package://robot_description/meshes/NEMA_24_2_1.stl" scale="0.001 0.001 0.001"/>
+    </geometry>
+    <material name="silver"/>
+  </visual>
+  <collision>
+    <origin rpy="0 0 0" xyz="-0.00348 -0.2275 -0.085"/>
+    <geometry>
+      <mesh filename="package://robot_description/meshes/NEMA_24_2_1.stl" scale="0.001 0.001 0.001"/>
+    </geometry>
+  </collision>
+</link>
+<link name="NEMA_24_3_1">
+  <inertial>
+    <origin rpy="0 0 0" xyz="7.65595409013553e-08 -0.04795079485405229 2.5568133205922106e-06"/>
     <mass value="2.4982959259379585"/>
     <inertia ixx="0.002718" ixy="0.0" ixz="0.0" iyy="0.001293" iyz="0.0" izz="0.002718"/>
   </inertial>
   <visual>
-    <origin rpy="0 0 0" xyz="-0.67155 0.00348 -0.820847"/>
-    <geometry>
-      <mesh filename="package://Robot_description/meshes/NEMA_24_v1__1__1.stl" scale="0.001 0.001 0.001"/>
-    </geometry>
-    <material name="silver"/>
-  </visual>
-  <collision>
-    <origin rpy="0 0 0" xyz="-0.67155 0.00348 -0.820847"/>
-    <geometry>
-      <mesh filename="package://Robot_description/meshes/NEMA_24_v1__1__1.stl" scale="0.001 0.001 0.001"/>
-    </geometry>
-  </collision>
-</link>
-<link name="NEMA_24_v1__2__1">
-  <inertial>
-    <origin rpy="0 0 0" xyz="-0.047950794854052514 -7.655954092217199e-08 3.0436810282141735e-06"/>
+    <origin rpy="0 0 0" xyz="-0.03848 -0.575 -0.085"/>
+    <geometry>
+      <mesh filename="package://robot_description/meshes/NEMA_24_3_1.stl" scale="0.001 0.001 0.001"/>
+    </geometry>
+    <material name="silver"/>
+  </visual>
+  <collision>
+    <origin rpy="0 0 0" xyz="-0.03848 -0.575 -0.085"/>
+    <geometry>
+      <mesh filename="package://robot_description/meshes/NEMA_24_3_1.stl" scale="0.001 0.001 0.001"/>
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
File: fusion_360_export/Robot_description/urdf/materials.xacro (robot description, xacro)
@@ -1,4 +1,4 @@
 <?xml version="1.0" ?>
-<robot name="Robot" xmlns:xacro="http://www.ros.org/wiki/xacro" >
+<robot name="robot" xmlns:xacro="http://www.ros.org/wiki/xacro" >
 <material name="silver">
   <color rgba="0.700 0.700 0.700 1.000"/>
