Commit message: added realsense plugin

File: fusion_360_export/robot_description/urdf/robot.xacro (robot description, xacro)
@@ -4,4 +4,5 @@
 <xacro:include filename="$(find robot_description)/urdf/robot.trans" />
 <xacro:include filename="$(find robot_description)/urdf/robot.gazebo" />
+<xacro:include filename="$(find robot_description)/urdf/_d435.urdf.xacro"/>
 <link name="base_link">
   <inertial>
@@ -444,4 +445,6 @@
   </collision>
 </link>
+<link name="RealSense_Camera_1"/>
+<!--
 <link name="RealSense_Camera_1">
   <inertial>
@@ -464,4 +467,10 @@
   </collision>
 </link>
+-->
+<!-- begin other fuckup -->
+<xacro:sensor_d435 parent="RealSense_Camera_1">
+	<!--<origin rpy="0 0 0" xyz="-0.44905 -0.09 -1.765675"/>-->
+	<origin rpy="0 0 0" xyz="0 0 0"/>
+</xacro:sensor_d435>
 <joint name="Rigid1" type="fixed">
   <origin rpy="0 0 0" xyz="0.0 0.075 -0.18"/>

Commit message: robot color added

File: fusion_360_export/robot_description/urdf/robot.xacro (robot description, xacro)
@@ -7,12 +7,12 @@
 <link name="base_link">
   <inertial>
-    <origin rpy="0 0 0" xyz="-1.4771468453599796e-05 -0.4394102251855798 -0.5105474620020639"/>
-    <mass value="90.2870635836035"/>
-    <inertia ixx="16.958749" ixy="-1.4e-05" ixz="-0.000256" iyy="10.456164" iyz="-0.360506" izz="18.430844"/>
+    <origin rpy="0 0 0" xyz="-0.00015399363028194057 -0.03925075208016042 0.2644524795806922"/>
+    <mass value="31.054157277051146"/>
+    <inertia ixx="3.596388" ixy="5e-06" ixz="-0.123996" iyy="5.832947" iyz="8.8e-05" izz="6.339272"/>
   </inertial>
   <visual>
     <origin rpy="0 0 0" xyz="0 0 0"/>
     <geometry>
-      <mesh filename="package://robot_description/meshes/base_link.stl" scale="0.001 0.001 0.001"/>
+      <mesh filename="package://robot_description/meshes/base_link.dae" scale="0.001 0.001 0.001"/>
     </geometry>
     <material name="silver"/>
@@ -21,5 +21,5 @@
     <origin rpy="0 0 0" xyz="0 0 0"/>
     <geometry>
-      <mesh filename="package://robot_description/meshes/base_link.stl" scale="0.001 0.001 0.001"/>
+      <mesh filename="package://robot_description/meshes/base_link.dae" scale="0.001 0.001 0.001"/>
     </geometry>
   </collision>
@@ -27,19 +27,19 @@
 <link name="arm_base_1">
   <inertial>
-    <origin rpy="0 0 0" xyz="-9.028631835610602e-14 -0.10852318160677443 0.07021749351752887"/>
+    <origin rpy="0 0 0" xyz="-0.10852294745565316 4.764549026911591e-07 0.07021749351752882"/>
     <mass value="2.9829690964186772"/>
-    <inertia ixx="0.024074" ixy="-0.0" ixz="-0.0" iyy="0.017973" iyz="-0.002884" izz="0.02919"/>
-  </inertial>
-  <visual>
-    <origin rpy="0 0 0" xyz="0.0 -0.075 0.18"/>
-    <geometry>
-      <mesh filename="package://robot_description/meshes/arm_base_1.stl" scale="0.001 0.001 0.001"/>
-    </geometry>
-    <material name="silver"/>
-  </visual>
-  <collision>
-    <origin rpy="0 0 0" xyz="0.0 -0.075 0.18"/>
-    <geometry>
-      <mesh filename="package://robot_description/meshes/arm_base_1.stl" scale="0.001 0.001 0.001"/>
+    <inertia ixx="0.017973" ixy="0.0" ixz="-0.002884" iyy="0.024074" iyz="0.0" izz="0.02919"/>
+  </inertial>
+  <visual>
+    <origin rpy="0 0 0" xyz="-0.514256 0.039266 -0.595"/>
+    <geometry>
+      <mesh filename="package://robot_description/meshes/arm_base_1.dae" scale="0.001 0.001 0.001"/>
+    </geometry>
+    <material name="silver"/>
+  </visual>
+  <collision>
+    <origin rpy="0 0 0" xyz="-0.514256 0.039266 -0.595"/>
+    <geometry>
+      <mesh filename="package://robot_description/meshes/arm_base_1.dae" scale="0.001 0.001 0.001"/>
     </geometry>
   </collision>
@@ -47,19 +47,19 @@
 <link name="stepper_joint_1">
   <inertial>
-    <origin rpy="0 0 0" xyz="0.007499999999999989 1.3028467193976212e-13 1.3877787807814457e-16"/>
-    <mass value="0.03498948817935604"/>
-    <inertia ixx="7e-06" ixy="0.0" ixz="0.0" iyy="4e-06" iyz="0.0" izz="4e-06"/>
-  </inertial>
-  <visual>
-    <origin rpy="0 0 0" xyz="-0.00348 -0.09 -0.085"/>
-    <geometry>
-      <mesh filename="package://robot_description/meshes/stepper_joint_1.stl" scale="0.001 0.001 0.001"/>
-    </geometry>
-    <material name="silver"/>
-  </visual>
-  <collision>
-    <origin rpy="0 0 0" xyz="-0.00348 -0.09 -0.085"/>
-    <geometry>
-      <mesh filename="package://robot_description/meshes/stepper_joint_1.stl" scale="0.001 0.001 0.001"/>
+    <origin rpy="0 0 0" xyz="2.341512516101929e-07 -0.007499523545187715 1.1102230246251565e-16"/>
+    <mass value="0.10172869711405369"/>
+    <inertia ixx="1.1e-05" ixy="0.0" ixz="-0.0" iyy="1.9e-05" iyz="-0.0" izz="1.1e-05"/>
+  </inertial>
+  <visual>
+    <origin rpy="0 0 0" xyz="-0.529256 0.042746 -0.86"/>
+    <geometry>
+      <mesh filename="package://robot_description/meshes/stepper_joint_1.dae" scale="0.001 0.001 0.001"/>
+    </geometry>
+    <material name="silver"/>
+  </visual>
+  <collision>
+    <origin rpy="0 0 0" xyz="-0.529256 0.042746 -0.86"/>
+    <geometry>
+      <mesh filename="package://robot_description/meshes/stepper_joint_1.dae" scale="0.001 0.001 0.001"/>
     </geometry>
   </collision>
@@ -67,19 +67,19 @@
 <link name="link_1_1">
   <inertial>
-    <origin rpy="0 0 0" xyz="-0.00750000000000001 0.2614820661654451 1.3877787807814457e-16"/>
+    <origin rpy="0 0 0" xyz="0.2614823003165665 0.0075004764548120065 0.0"/>
     <mass value="1.2422891158221263"/>
-    <inertia ixx="0.03033" ixy="0.0" ixz="0.0" iyy="0.000414" iyz="-0.0" izz="0.029962"/>
-  </inertial>
-  <visual>
-    <origin rpy="0 0 0" xyz="-0.00348 -0.09 -0.085"/>
-    <geometry>
-      <mesh filename="package://robot_description/meshes/link_1_1.stl" scale="0.001 0.001 0.001"/>
-    </geometry>
-    <material name="silver"/>
-  </visual>
-  <collision>
-    <origin rpy="0 0 0" xyz="-0.00348 -0.09 -0.085"/>
-    <geometry>
-      <mesh filename="package://robot_description/meshes/link_1_1.stl" scale="0.001 0.001 0.001"/>
+    <inertia ixx="0.000414" ixy="0.0" ixz="0.0" iyy="0.03033" iyz="0.0" izz="0.029962"/>
+  </inertial>
+  <visual>
+    <origin rpy="0 0 0" xyz="-0.529256 0.042746 -0.86"/>
+    <geometry>
+      <mesh filename="package://robot_description/meshes/link_1_1.dae" scale="0.001 0.001 0.001"/>
+    </geometry>
+    <material name="silver"/>
+  </visual>
+  <collision>
+    <origin rpy="0 0 0" xyz="-0.529256 0.042746 -0.86"/>
+    <geometry>
+      <mesh filename="package://robot_description/meshes/link_1_1.dae" scale="0.001 0.001 0.001"/>
     </geometry>
   </collision>
@@ -87,19 +87,19 @@
 <link name="link_2_1">
   <inertial>
-    <origin rpy="0 0 0" xyz="0.026213672668365277 0.017799785433927795 1.3877787807814457e-16"/>
+    <origin rpy="0 0 0" xyz="0.017800019585049176 -0.026213196213553565 0.0"/>
     <mass value="0.8743627585315773"/>
-    <inertia ixx="0.000992" ixy="-8.4e-05" ixz="0.0" iyy="0.000864" iyz="0.0" izz="0.001253"/>
-  </inertial>
-  <visual>
-    <origin rpy="0 0 0" xyz="-0.00348 -0.605 -0.085"/>
-    <geometry>
-      <mesh filename="package://robot_description/meshes/link_2_1.stl" scale="0.001 0.001 0.001"/>
-    </geometry>
-    <material name="silver"/>
-  </visual>
-  <collision>
-    <origin rpy="0 0 0" xyz="-0.00348 -0.605 -0.085"/>
-    <geometry>
-      <mesh filename="package://robot_description/meshes/link_2_1.stl" scale="0.001 0.001 0.001"/>
+    <inertia ixx="0.000864" ixy="8.4e-05" ixz="0.0" iyy="0.000992" iyz="-0.0" izz="0.001253"/>
+  </inertial>
+  <visual>
+    <origin rpy="0 0 0" xyz="-1.044256 0.042746 -0.86"/>
+    <geometry>
+      <mesh filename="package://robot_description/meshes/link_2_1.dae" scale="0.001 0.001 0.001"/>
+    </geometry>
+    <material name="silver"/>
+  </visual>
+  <collision>
+    <origin rpy="0 0 0" xyz="-1.044256 0.042746 -0.86"/>
+    <geometry>
+      <mesh filename="package://robot_description/meshes/link_2_1.dae" scale="0.001 0.001 0.001"/>
     </geometry>
   </collision>
@@ -107,19 +107,19 @@
 <link name="link_3_1">
   <inertial>
-    <origin rpy="0 0 0" xyz="0.02499852381758487 0.1769222136151417 3.885780586188048e-16"/>
+    <origin rpy="0 0 0" xyz="0.17692244776626231 -0.02499804736277332 3.3306690738754696e-16"/>
     <mass value="1.5478777520934175"/>
-    <inertia ixx="0.032303" ixy="-0.002603" ixz="0.0" iyy="0.001209" iyz="0.0" izz="0.032482"/>
-  </inertial>
-  <visual>
-    <origin rpy="0 0 0" xyz="-0.03848 -0.675 -0.085"/>
-    <geometry>
-      <mesh filename="package://robot_description/meshes/link_3_1.stl" scale="0.001 0.001 0.001"/>
-    </geometry>
-    <material name="silver"/>
-  </visual>
-  <collision>
-    <origin rpy="0 0 0" xyz="-0.03848 -0.675 -0.085"/>
-    <geometry>
-      <mesh filename="package://robot_description/meshes/link_3_1.stl" scale="0.001 0.001 0.001"/>
+    <inertia ixx="0.001209" ixy="0.002603" ixz="-0.0" iyy="0.032303" iyz="0.0" izz="0.032482"/>
+  </inertial>
+  <visual>
+    <origin rpy="0 0 0" xyz="-1.114256 0.077746 -0.86"/>
+    <geometry>
+      <mesh filename="package://robot_description/meshes/link_3_1.dae" scale="0.001 0.001 0.001"/>
+    </geometry>
+    <material name="silver"/>
+  </visual>
+  <collision>
+    <origin rpy="0 0 0" xyz="-1.114256 0.077746 -0.86"/>
+    <geometry>
+      <mesh filename="package://robot_description/meshes/link_3_1.dae" scale="0.001 0.001 0.001"/>
     </geometry>
   </collision>
@@ -127,39 +127,19 @@
 <link name="link_end_1">
   <inertial>
-    <origin rpy="0 0 0" xyz="-0.03379678599677132 0.011579118062804872 4.163336342344337e-16"/>
+    <origin rpy="0 0 0" xyz="0.011579352213925143 0.033797262451582544 1.1102230246251565e-16"/>
     <mass value="1.063293416063342"/>
-    <inertia ixx="0.000747" ixy="7.6e-05" ixz="0.0" iyy="0.00115" iyz="-0.0" izz="0.001353"/>
-  </inertial>
-  <visual>
-    <origin rpy="0 0 0" xyz="-0.06848 -1.13 -0.085"/>
-    <geometry>
-      <mesh filename="package://robot_description/meshes/link_end_1.stl" scale="0.001 0.001 0.001"/>
-    </geometry>
-    <material name="silver"/>
-  </visual>
-  <collision>
-    <origin rpy="0 0 0" xyz="-0.06848 -1.13 -0.085"/>
-    <geometry>
-      <mesh filename="package://robot_description/meshes/link_end_1.stl" scale="0.001 0.001 0.001"/>
-    </geometry>
-  </collision>
-</link>
-<link name="NEMA_24_1_1">
-  <inertial>
-    <origin rpy="0 0 0" xyz="-2.5568133205304072e-06 7.655954109564433e-08 0.047950794854052264"/>
-    <mass value="2.4982959259379585"/>
-    <inertia ixx="0.002718" ixy="-0.0" ixz="0.0" iyy="0.002718" iyz="-0.0" izz="0.001293"/>
-  </inertial>
-  <visual>
-    <origin rpy="0 0 0" xyz="-0.0 0.125 0.12"/>
-    <geometry>
-      <mesh filename="package://robot_description/meshes/NEMA_24_1_1.stl" scale="0.001 0.001 0.001"/>
-    </geometry>
-    <material name="silver"/>
-  </visual>
-  <collision>
-    <origin rpy="0 0 0" xyz="-0.0 0.125 0.12"/>
-    <geometry>
-      <mesh filename="package://robot_description/meshes/NEMA_24_1_1.stl" scale="0.001 0.001 0.001"/>
+    <inertia ixx="0.00115" ixy="-7.6e-05" ixz="-0.0" iyy="0.000747" iyz="0.0" izz="0.001353"/>
+  </inertial>
+  <visual>
+    <origin rpy="0 0 0" xyz="-1.569256 0.107746 -0.86"/>
+    <geometry>
+      <mesh filename="package://robot_description/meshes/link_end_1.dae" scale="0.001 0.001 0.001"/>
+    </geometry>
+    <material name="silver"/>
+  </visual>
+  <collision>
+    <origin rpy="0 0 0" xyz="-1.569256 0.107746 -0.86"/>
+    <geometry>
+      <mesh filename="package://robot_description/meshes/link_end_1.dae" scale="0.001 0.001 0.001"/>
     </geometry>
   </collision>
@@ -167,39 +147,39 @@
 <link name="NEMA_24_2_1">
   <inertial>
-    <origin rpy="0 0 0" xyz="0.04795079485405226 7.655954106788876e-08 2.556813320619966e-06"/>
-    <mass value="2.4982959259379585"/>
-    <inertia ixx="0.001293" ixy="-0.0" ixz="-0.0" iyy="0.002718" iyz="0.0" izz="0.002718"/>
-  </inertial>
-  <visual>
-    <origin rpy="0 0 0" xyz="-0.00348 -0.2275 -0.085"/>
-    <geometry>
-      <mesh filename="package://robot_description/meshes/NEMA_24_2_1.stl" scale="0.001 0.001 0.001"/>
-    </geometry>
-    <material name="silver"/>
-  </visual>
-  <collision>
-    <origin rpy="0 0 0" xyz="-0.00348 -0.2275 -0.085"/>
-    <geometry>
-      <mesh filename="package://robot_description/meshes/NEMA_24_2_1.stl" scale="0.001 0.001 0.001"/>
-    </geometry>
-  </collision>
-</link>
-<link name="NEMA_24_3_1">
-  <inertial>
-    <origin rpy="0 0 0" xyz="7.65595409013553e-08 -0.04795079485405229 2.5568133205922106e-06"/>
+    <origin rpy="0 0 0" xyz="3.107106621991207e-07 -0.04795031839924011 2.5568133203979215e-06"/>
     <mass value="2.4982959259379585"/>
     <inertia ixx="0.002718" ixy="0.0" ixz="0.0" iyy="0.001293" iyz="0.0" izz="0.002718"/>
   </inertial>
   <visual>
-    <origin rpy="0 0 0" xyz="-0.03848 -0.575 -0.085"/>
-    <geometry>
-      <mesh filename="package://robot_description/meshes/NEMA_24_3_1.stl" scale="0.001 0.001 0.001"/>
-    </geometry>
-    <material name="silver"/>
-  </visual>
-  <collision>
-    <origin rpy="0 0 0" xyz="-0.03848 -0.575 -0.085"/>
-    <geometry>
-      <mesh filename="package://robot_description/meshes/NEMA_24_3_1.stl" scale="0.001 0.001 0.001"/>
+    <origin rpy="0 0 0" xyz="-0.666756 0.042746 -0.86"/>
+    <geometry>
+      <mesh filename="package://robot_description/meshes/NEMA_24_2_1.dae" scale="0.001 0.001 0.001"/>
+    </geometry>
+    <material name="silver"/>
+  </visual>
+  <collision>
+    <origin rpy="0 0 0" xyz="-0.666756 0.042746 -0.86"/>
+    <geometry>
+      <mesh filename="package://robot_description/meshes/NEMA_24_2_1.dae" scale="0.001 0.001 0.001"/>
+    </geometry>
+  </collision>
+</link>
+<link name="NEMA_24_3_1">
+  <inertial>
+    <origin rpy="0 0 0" xyz="-0.04744967584155013 4.039331734789764e-07 3.008172847374091e-06"/>
+    <mass value="0.9071303592190116"/>
+    <inertia ixx="0.000445" ixy="-0.0" ixz="0.0" iyy="0.000995" iyz="-0.0" izz="0.000995"/>
+  </inertial>
+  <visual>
+    <origin rpy="0 0 0" xyz="-1.014256 0.077746 -0.86"/>
+    <geometry>
+      <mesh filename="package://robot_description/meshes/NEMA_24_3_1.dae" scale="0.001 0.001 0.001"/>
+    </geometry>
+    <material name="silver"/>
+  </visual>
+  <collision>
+    <origin rpy="0 0 0" xyz="-1.014256 0.077746 -0.86"/>
+    <geometry>
+      <mesh filename="package://robot_description/meshes/NEMA_24_3_1.dae" scale="0.001 0.001 0.001"/>
     </geometry>
   </collision>
@@ -207,19 +187,19 @@
 <link name="NEMA_24_4_1">
   <inertial>
-    <origin rpy="0 0 0" xyz="-7.655954063073844e-08 0.0009492051459477624 -0.029802556813320228"/>
-    <mass value="2.4982959259379585"/>
-    <inertia ixx="0.002718" ixy="-0.0" ixz="0.0" iyy="0.001293" iyz="-0.0" izz="0.002718"/>
-  </inertial>
-  <visual>
-    <origin rpy="0 0 0" xyz="-0.03598 -0.625 -0.055"/>
-    <geometry>
-      <mesh filename="package://robot_description/meshes/NEMA_24_4_1.stl" scale="0.001 0.001 0.001"/>
-    </geometry>
-    <material name="silver"/>
-  </visual>
-  <collision>
-    <origin rpy="0 0 0" xyz="-0.03598 -0.625 -0.055"/>
-    <geometry>
-      <mesh filename="package://robot_description/meshes/NEMA_24_4_1.stl" scale="0.001 0.001 0.001"/>
+    <origin rpy="0 0 0" xyz="0.0014503241584495896 5.489764498406435e-07 -0.029803008172847645"/>
+    <mass value="0.9071303592190116"/>
+    <inertia ixx="0.000445" ixy="0.0" ixz="-0.0" iyy="0.000995" iyz="-0.0" izz="0.000995"/>
+  </inertial>
+  <visual>
+    <origin rpy="0 0 0" xyz="-1.064256 0.075246 -0.83"/>
+    <geometry>
+      <mesh filename="package://robot_description/meshes/NEMA_24_4_1.dae" scale="0.001 0.001 0.001"/>
+    </geometry>
+    <material name="silver"/>
+  </visual>
+  <collision>
+    <origin rpy="0 0 0" xyz="-1.064256 0.075246 -0.83"/>
+    <geometry>
+      <mesh filename="package://robot_description/meshes/NEMA_24_4_1.dae" scale="0.001 0.001 0.001"/>
     </geometry>
   </collision>
@@ -227,19 +207,19 @@
 <link name="gripper_base_1">
   <inertial>
-    <origin rpy="0 0 0" xyz="-8.738046848588699e-10 0.03673655788581898 1.1906876873357675e-10"/>
-    <mass value="1.1315792783817065"/>
-    <inertia ixx="0.001126" ixy="0.0" ixz="-0.0" iyy="0.001318" iyz="-0.0" izz="0.001126"/>
-  </inertial>
-  <visual>
-    <origin rpy="0 0 0" xyz="-0.02848 -1.18 -0.085"/>
-    <geometry>
-      <mesh filename="package://robot_description/meshes/gripper_base_1.stl" scale="0.001 0.001 0.001"/>
-    </geometry>
-    <material name="silver"/>
-  </visual>
-  <collision>
-    <origin rpy="0 0 0" xyz="-0.02848 -1.18 -0.085"/>
-    <geometry>
-      <mesh filename="package://robot_description/meshes/gripper_base_1.stl" scale="0.001 0.001 0.001"/>
+    <origin rpy="0 0 0" xyz="0.03673679203693969 4.773286157999657e-07 1.1906853281118401e-10"/>
+    <mass value="0.3892056116726888"/>
+    <inertia ixx="0.000453" ixy="-0.0" ixz="-0.0" iyy="0.000387" iyz="0.0" izz="0.000387"/>
+  </inertial>
+  <visual>
+    <origin rpy="0 0 0" xyz="-1.619256 0.067746 -0.86"/>
+    <geometry>
+      <mesh filename="package://robot_description/meshes/gripper_base_1.dae" scale="0.001 0.001 0.001"/>
+    </geometry>
+    <material name="silver"/>
+  </visual>
+  <collision>
+    <origin rpy="0 0 0" xyz="-1.619256 0.067746 -0.86"/>
+    <geometry>
+      <mesh filename="package://robot_description/meshes/gripper_base_1.dae" scale="0.001 0.001 0.001"/>
     </geometry>
   </collision>
@@ -247,19 +227,19 @@
 <link name="gripper_finger_1_1">
   <inertial>
-    <origin rpy="0 0 0" xyz="-3.2830821047880043e-10 0.022979968590664424 0.004865333770814467"/>
-    <mass value="0.07511526055866109"/>
-    <inertia ixx="1.7e-05" ixy="0.0" ixz="-0.0" iyy="3e-06" iyz="-0.0" izz="1.8e-05"/>
-  </inertial>
-  <visual>
-    <origin rpy="0 0 0" xyz="-0.02848 -1.2645 -0.1175"/>
-    <geometry>
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