Commit message: holonomic movement fix

File: robot_description/urdf/robot.xacro (robot description, xacro)
@@ -5,4 +5,10 @@
 <xacro:include filename="$(find robot_description)/urdf/robot.gazebo" />
 <xacro:include filename="$(find robot_description)/urdf/_d435.urdf.xacro"/>
+<link name="base_frame"></link>
+<joint name="base_frame_joint" type="fixed">
+  <origin xyz="0 0 0" rpy="0 0 0" />
+  <parent link="base_frame"/>
+  <child link="base_link"/>
+</joint>
 <link name="base_link">
   <inertial>
@@ -285,4 +291,5 @@
   </collision>
 </link>
+<!--WHEELS-->
 <link name="wheel_front_left_1">
   <inertial>
