Commit message: robot desc. changes

File: robot_description/urdf/_d435.gazebo.xacro (robot description, xacro)
@@ -27,6 +27,6 @@
           <horizontal_fov>${69.4*deg_to_rad}</horizontal_fov>
           <image>
-            <width>1920</width>
-            <height>1080</height>
+            <width>1280</width>
+            <height>720</height>
             <format>RGB_INT8</format>
           </image>
@@ -63,5 +63,5 @@
           </noise>
         </camera>
-        <always_on>1</always_on>
+        <always_on>0</always_on>
         <update_rate>90</update_rate>
         <visualize>0</visualize>
@@ -85,5 +85,5 @@
           </noise>
         </camera>
-        <always_on>1</always_on>
+        <always_on>0</always_on>
         <update_rate>90</update_rate>
         <visualize>0</visualize>
@@ -107,5 +107,5 @@
         </camera>
         <always_on>1</always_on>
-        <update_rate>90</update_rate>
+        <update_rate>30</update_rate>
         <visualize>0</visualize>
       </sensor>
@@ -131,5 +131,5 @@
       	<rangeMinDepth>0.2</rangeMinDepth>
       	<rangeMaxDepth>10.0</rangeMaxDepth>
-      	<pointCloud>false</pointCloud>
+      	<pointCloud>true</pointCloud>
       	<pointCloudTopicName>depth/points</pointCloudTopicName>
       	<pointCloudCutoff>0.5</pointCloudCutoff>

File: robot_description/urdf/robot.xacro (robot description, xacro)
@@ -51,5 +51,5 @@
   </collision>
 </link>
-<link name="stepper_joint_1">
+<!-- <link name="stepper_joint_1">
   <inertial>
     <origin rpy="0 0 0" xyz="2.341512516101929e-07 -0.007499523545187715 1.1102230246251565e-16"/>
@@ -290,5 +290,5 @@
     </geometry>
   </collision>
-</link>
+</link> -->
 <!--WHEELS-->
 <link name="wheel_front_left_1">
@@ -428,5 +428,5 @@
   </collision>
 </link>
-<link name="NEMA_34_1">
+<!-- <link name="NEMA_34_1">
   <inertial>
     <origin rpy="0 0 0" xyz="-1.8231621852216051e-06 -0.07677876842578721 -1.1102230246251565e-16"/>
@@ -447,5 +447,5 @@
     </geometry>
   </collision>
-</link>
+</link> -->
 <!--
 <link name="RealSense_Camera_1">
@@ -474,5 +474,5 @@
 	<origin rpy="0 0 0" xyz="0 0 0"/>
 </xacro:sensor_d435>
-<link name="NEMA_24_1_1">
+<!-- <link name="NEMA_24_1_1">
   <inertial>
     <origin rpy="0 0 0" xyz="3.1071066247667645e-07 3.0332681329736655e-06 0.04795079485405218"/>
@@ -573,5 +573,5 @@
     </geometry>
   </collision>
-</link>
+</link> -->
 <joint name="Rigid1" type="fixed">
   <origin rpy="0 0 0" xyz="0.514256 -0.039266 0.595"/>
@@ -579,4 +579,5 @@
   <child link="arm_base_1"/>
 </joint>
+<!--
 <joint name="Rigid4" type="fixed">
   <origin rpy="0 0 0" xyz="0.0 0.03652 0.0"/>
@@ -645,5 +646,5 @@
   <child link="gripper_finger_3_1"/>
   <axis xyz="0.0 0.5 0.866025"/>
-</joint>
+</joint> -->
 <joint name="wheel_joint_front_left" type="continuous">
   <origin rpy="0 0 0" xyz="0.389785 0.351556 0.072882"/>
@@ -681,9 +682,10 @@
   <axis xyz="-0.0 0.0 -1.0"/>
 </joint>
+<!--
 <joint name="Rigid28" type="fixed">
   <origin rpy="0 0 0" xyz="0.09 -0.04 0.085"/>
   <parent link="base_turnable_1"/>
   <child link="NEMA_34_1"/>
-</joint>
+</joint> -->
 <joint name="camera_revolute" type="continuous">
   <origin rpy="0 0 0" xyz="0.005 0.09 0.629827"/>
@@ -692,4 +694,5 @@
   <axis xyz="-0.0 0.0 -1.0"/>
 </joint>
+<!--
 <joint name="Rigid30" type="fixed">
   <origin rpy="0 0 0" xyz="-0.2 0.0 0.06"/>
@@ -716,4 +719,4 @@
   <parent link="base_link"/>
   <child link="DistanceSensor_back_1"/>
-</joint>
+</joint> -->
 </robot>
